File: morro-bay/PCB_Morro_Bay/ExternalADC.sch (KiCad schematic (older format))
At the start: 89 parts, among them SW4 INPUT_RANGE_SEL_3, U10 LM2902, U11 LM2902, U12 LM2902, U26 ADS114S08BIPBSR

Commit message: Export final gerbers for MB
Parts:
- R100, R102, R104, R110, R111, R98: Digikey https://www.digikey.ca/product-detail/en/stackpole-electron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 -> https://www.digikey.ca/en/products/detail/yageo/RC0603FR-07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; Part Number RMCF0603FT47R0 -> RC0603FR-0747RL
- R106, R107, R108, R109, R75, R77, R79, R81, R87, R89, R91, R93: Digikey https://www.digikey.ca/product-detail/en/panasonic-electron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 -> https://www.digikey.ca/en/products/detail/panasonic-electro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; Part Number ERJ-PB3B1003V -> ERA-3AEB104V
