File: morro-bay/PCB_Morro_Bay/PCB_Morro_Bay.kicad_pcb (KiCad board)
At the start: 2 copper layers, 341 parts, among them J1 POWER, J10 Conn_01x04, J11 Conn_01x04, J12 Conn_01x04, J13 Conn_01x04, J14 Conn_01x04, J15 Conn_01x04, J16 Conn_01x04, J17 Conn_01x04, J18 Conn_01x04, J19 Conn_01x04, J2 CAN, J20 Conn_01x04, J21 Conn_01x04, J22 Conn_01x04, J23 POWER_OUT, J24 Conn_01x04, J25 Conn_01x04, J26 Conn_01x04, J27 Conn_01x04, J28 Conn_01x04, J29 Conn_01x04, J3 Conn_01x04, J30 Conn_01x04, J31 Conn_01x04, J32 Conn_01x04, J33 Conn_01x04, J34 Conn_01x04, J35 Conn_01x04, J36 SWD, J37 GPIO, J38 USB_B, J39 ESERCOM, J4 Conn_01x04, J5 Conn_01x04, J6 Conn_01x04, J7 Conn_01x04, J8 Conn_01x04, J9 Conn_01x04, SW1 INPUT_RANGE_SEL_1, SW2 INPUT_RANGE_SEL_2, SW3 RESET, SW4 INPUT_RANGE_SEL_3, U1 MCP2515-xSO, U10 LM2902, U11 LM2902, U12 LM2902, U13 V7805-2000R, U2 SN65HVD232, U26 ADS114S08BIPBSR, U3 AZ1117-3.3, U4 ATSAMD21J18A-AU, U5 LM2902, U6 LM2902, U7 LM2902, U8 LM2902, U9 LM2902, Y1 8MHz, Y2 30MHz, Y3 32.768kHz

Commit message: Fix values of C7 and C8
Parts:
- C36, R17: moved to F.Cu
- C7: value 1uF -> 10uF
- C8: value 1uF -> 22uF; footprint Capacitor_SMD:C_0603_1608Metric_Pad1.05x0.95mm_HandSolder -> Capacitor_SMD:C_0805_2012Metric_Pad1.15x1.40mm_HandSolder
- J10: value Conn_01x04 -> 5V_12_8
- J11: value Conn_01x04 -> 5V_12_9
- J12: value Conn_01x04 -> 5V_12_10
- J13: value Conn_01x04 -> 5V_12_11
- J14: value Conn_01x04 -> 5V_12_12
- J15: value Conn_01x04 -> 5V_12_13
- J16: value Conn_01x04 -> 5V_12_14
- J17: value Conn_01x04 -> 10V_12_1
- J18: value Conn_01x04 -> 10V_12_2
- J19: value Conn_01x04 -> 10V_12_3
- J20: value Conn_01x04 -> 10V_12_4
- J21: value Conn_01x04 -> 10V_12_5
- J22: value Conn_01x04 -> 10V_12_6
- J24: value Conn_01x04 -> 5V_16_1
- J25: value Conn_01x04 -> 5V_16_2
- J26: value Conn_01x04 -> 5V_16_3
- J27: value Conn_01x04 -> 5V_16_4
- J28: value Conn_01x04 -> 10V_16_1
- J29: value Conn_01x04 -> 10V_16_2
- J3: value Conn_01x04 -> 5V_12_1
- J30: value Conn_01x04 -> 10V_16_3
- J31: value Conn_01x04 -> 10V_16_4
- J32: value Conn_01x04 -> 5V_16_5
- J33: value Conn_01x04 -> 5V_16_6
- J34: value Conn_01x04 -> 5V_16_7
- J35: value Conn_01x04 -> 5V_16_8
- J4: value Conn_01x04 -> 5V_12_2
- J5: value Conn_01x04 -> 5V_12_3
- J6: value Conn_01x04 -> 5V_12_4
- J7: value Conn_01x04 -> 5V_12_5
- J8: value Conn_01x04 -> 5V_12_6
- J9: value Conn_01x04 -> 5V_12_7
- R120, R121, R122, R123: moved to B.Cu
- moved J35 496.4 mm to (64.8, 129.8), turned to 180 degrees
- moved TP40 491.6 mm to (62.5, 112.8), turned to 270 degrees
- moved R92 485.6 mm to (65.8, 113.2), turned to 90 degrees
- moved R109 481.2 mm to (68.0, 113.2), turned to 270 degrees
- moved J34 465.3 mm to (79.8, 129.8), turned to 180 degrees
- moved TP39 459.9 mm to (77.5, 112.8), turned to 270 degrees
- moved R90 453.8 mm to (80.8, 113.2), turned to 90 degrees
- moved R108 449.5 mm to (83.0, 113.2), turned to 270 degrees
- moved J33 434.4 mm to (94.8, 129.8), turned to 180 degrees
- moved TP38 428.2 mm to (92.5, 112.8), turned to 270 degrees
- moved R88 422.2 mm to (95.8, 113.2), turned to 90 degrees
- moved R107 417.9 mm to (98.0, 113.2), turned to 270 degrees
- moved J32 403.7 mm to (109.8, 129.8), turned to 180 degrees
- moved TP37 396.8 mm to (107.5, 112.8), turned to 270 degrees
- moved R86 390.9 mm to (110.8, 113.2), turned to 90 degrees
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Connections:
- C66 pad 1: +3V3 -> Net-(C66-Pad1)
- C66 pad 2: GND -> Net-(C66-Pad2)
Other:
- board outline added: 250 x 100 mm

Commit message: Layout
Parts:
- moved C48 95.9 mm to (91.2, 98.5)
- moved C49 95.9 mm to (87.0, 101.5)
- moved R43 95.9 mm to (87.0, 98.5)
- moved R44 95.9 mm to (82.8, 101.5)
- moved U7 82.5 mm to (72.2, 87.0)
- moved R41 80.9 mm to (66.0, 83.2)
- moved C47 76.5 mm to (62.2, 89.8)
- moved C24 75.5 mm to (72.2, 93.2), turned to 180 degrees
- moved C46 73.1 mm to (62.2, 83.2)
- moved R42 71.4 mm to (66.0, 89.8)
- moved R30 26.8 mm to (66.0, 74.8)
- moved R32 22.2 mm to (78.5, 68.2), turned to 180 degrees
- moved C44 11.4 mm to (82.2, 74.8), turned to 180 degrees
- moved C22 0.25 mm to (72.2, 63.2)
- moved C23 0.25 mm to (72.2, 78.2)
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
Commit message: Much layout
Parts:
- U13: moved to B.Cu
- moved C54 276.0 mm to (248.8, 77.5), turned to 270 degrees
- moved R61 272.9 mm to (248.8, 81.2), turned to 270 degrees
- moved C52 272.8 mm to (247.2, 59.8), turned to 180 degrees
- moved C53 271.4 mm to (247.2, 53.2), turned to 180 degrees
- moved R55 267.9 mm to (243.5, 59.8), turned to 180 degrees
- moved C70 266.8 mm to (77.2, 99.8)
- moved C71 266.3 mm to (77.2, 106.2)
- moved C55 266.1 mm to (242.2, 77.5), turned to 270 degrees
- moved U9 263.5 mm to (245.0, 87.5), turned to 270 degrees
- moved D1 263.5 mm to (62.2, 55.2), turned to 180 degrees
- moved R62 263.3 mm to (242.2, 81.2), turned to 270 degrees
- moved R56 261.0 mm to (243.5, 53.2), turned to 180 degrees
- moved D3 259.6 mm to (82.2, 61.8)
- moved R114 259.4 mm to (81.0, 99.8)
- moved R115 258.9 mm to (81.0, 106.2)
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
Commit message: Start routing
Parts:
- C1, C2, C30, C31, C33, C34, C35, C58, C59, C6, C60, C61, C62, C63, C64, C65, C67, C68, C69, C70, C71, C9, D23, D24, D25, D26, D27, D28, D29, D30, D31, D32, D33, D34, D35, D36, JP1, R1, R100, R102, R104, R110, R111, R112, R113, R114, R115, R116, R117, R2, R3, R6, R8, R82, R83, R84, R85, R94, R95, R96, R97, R98, TP1, TP2, TP3, TP4, U1, U10, U11, U12, U2, U26, Y1: moved to B.Cu
- moved R8 266.6 mm to (55.2, 85.8), turned to 90 degrees
- moved TP1 261.2 mm to (42.5, 74.2), turned to 180 degrees
- moved D35 261.0 mm to (43.0, 78.8), turned to 180 degrees
- moved D36 261.0 mm to (47.0, 78.8), turned to 180 degrees
- moved R116 261.0 mm to (43.0, 76.8), turned to 180 degrees
- moved R117 261.0 mm to (47.0, 76.8), turned to 180 degrees
- moved TP2 260.7 mm to (47.5, 74.2), turned to 180 degrees
- moved R1 259.0 mm to (61.0, 85.8), turned to 90 degrees
- moved R2 256.6 mm to (62.8, 85.8), turned to 90 degrees
- moved R3 254.2 mm to (64.5, 85.8), turned to 90 degrees
- moved U1 250.1 mm to (59.0, 77.8), turned to 270 degrees
- moved R4 248.2 mm to (57.0, 69.5), turned to 270 degrees
- moved R5 245.8 mm to (58.8, 69.5), turned to 270 degrees
- moved R6 244.6 mm to (43.8, 69.2), turned to 270 degrees
- moved TP4 244.5 mm to (39.5, 68.5)
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Connections:
- C66 pad 1: Net-(C66-Pad1) -> +3V3
- C66 pad 2: Net-(C66-Pad2) -> GND
Routing:
- net GND: track 0.00 -> 157.6 mm
- net /CAN_TX: track 0.00 -> 25.5 mm
- net /CAN_XTAL_2: track 0.00 -> 23.8 mm
- net /CAN_RX: track 0.00 -> 18.8 mm
- net /USB_D-: track 0.00 -> 13.9 mm
- net /CANL: track 0.00 -> 13.2 mm
- net /CANH: track 0.00 -> 13.1 mm
- net /CAN_XTAL_1: track 0.00 -> 11.7 mm
- net /USB_D+: track 0.00 -> 8.33 mm
- net Net-(H1-Pad1): track 0.00 -> 7.45 mm
- net Net-(H4-Pad1): track 0.00 -> 7.45 mm
- net Net-(H2-Pad1): track 0.00 -> 7.45 mm
- net Net-(H3-Pad1): track 0.00 -> 7.45 mm
- net 5V_IN_16: track 0.00 -> 6.49 mm
- net 5V_IN_21: track 0.00 -> 6.49 mm
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
Commit message: Routing and layout work
Parts:
- C22, C23, C24, C36, C37, C38, C39, C42, C43, C44, C45, C46, C47, C48, C49, D1, D10, D11, D12, D2, D3, D4, D5, D6, D7, D8, D9, R17, R18, R19, R20, R29, R30, R31, R32, R41, R42, R43, R44, U5, U6, U7: moved to B.Cu
- moved D2 22.2 mm to (82.2, 52.0), turned to 0 degrees
- moved D3 22.2 mm to (62.2, 52.0), turned to 180 degrees
- moved C36 21.3 mm to (82.2, 60.5), turned to 180 degrees
- moved C39 21.3 mm to (62.2, 60.5), turned to 0 degrees
- moved C37 20.8 mm to (82.2, 54.0), turned to 180 degrees
- moved C38 20.8 mm to (62.2, 54.0), turned to 0 degrees
- moved D1 20.3 mm to (82.2, 58.5), turned to 0 degrees
- moved D4 20.3 mm to (62.2, 58.5), turned to 180 degrees
- moved R17 14.5 mm to (78.5, 60.5), turned to 180 degrees
- moved R20 14.5 mm to (66.0, 60.5), turned to 0 degrees
- moved R18 13.8 mm to (78.5, 54.0), turned to 180 degrees
- moved R19 13.8 mm to (66.0, 54.0), turned to 0 degrees
- moved C24 12.0 mm to (192.2, 51.0)
- moved D10 9.50 mm to (182.2, 52.2)
- moved D11 9.50 mm to (202.2, 52.2)
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Connections:
- U4 pad 10: SAMD_ADC_10 -> SAMD_ADC_11
- U4 pad 11: SAMD_ADC_11 -> SAMD_ADC_10
- U4 pad 12: SAMD_ADC_12 -> SAMD_ADC_9
- U4 pad 13: SAMD_ADC_13 -> SAMD_ADC_8
- U4 pad 14: SAMD_ADC_14 -> SAMD_ADC_7
- U4 pad 15: SAMD_ADC_15 -> SAMD_ADC_6
- U4 pad 16: SAMD_ADC_16 -> SAMD_ADC_5
- U4 pad 17: SAMD_ADC_17 -> SAMD_ADC_4
- U4 pad 18: SAMD_ADC_18 -> SAMD_ADC_3
- U4 pad 19: SAMD_ADC_19 -> SAMD_ADC_2
- U4 pad 20: SAMD_ADC_20 -> SAMD_ADC_1
- U4 pad 3: SAMD_ADC_5 -> SAMD_ADC_16
- U4 pad 4: SAMD_ADC_6 -> SAMD_ADC_15
- U4 pad 5: SAMD_ADC_7 -> SAMD_ADC_14
- U4 pad 6: SAMD_ADC_8 -> SAMD_ADC_13
- U4 pad 61: SAMD_ADC_1 -> SAMD_ADC_20
- U4 pad 62: SAMD_ADC_2 -> SAMD_ADC_19
- U4 pad 63: SAMD_ADC_3 -> SAMD_ADC_18
- U4 pad 64: SAMD_ADC_4 -> SAMD_ADC_17
- U4 pad 9: SAMD_ADC_9 -> SAMD_ADC_12
Routing:
- net GND: track 157.6 -> 178.0 mm
- net Net-(R71-Pad2): track 0.00 -> 12.8 mm
- net /LED_1: track 0.00 -> 12.5 mm
- net +3V3: track 2.40 -> 14.4 mm
- net /SAMD_XTAL2_2: track 0.00 -> 10.2 mm
- net /LED_2: track 0.00 -> 9.38 mm
- net /SAMD_XTAL2_1: track 0.00 -> 9.20 mm
- net /SAMD_nRESET: track 0.00 -> 7.02 mm
- net +3.3VA: track 0.00 -> 4.85 mm
- net /SWCLK: track 0.00 -> 4.04 mm
- net Net-(C19-Pad1): track 0.00 -> 3.42 mm
- net /AnalogInput/IN_3_BUFFERED: track 4.03 -> 1.27 mm
- net /AnalogInput/IN_2_BUFFERED: track 4.03 -> 1.27 mm
- net /AnalogInput/IN_4_BUFFERED: track 3.97 -> 1.35 mm
- net /AnalogInput/IN_1_BUFFERED: track 3.97 -> 1.35 mm
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
Commit message: Routed some things
Parts:
- C22, C23, C24, C30, C31, C36, C37, C38, C39, C42, C43, C44, C45, C46, C47, C48, C49, C58, C59, C60, C61, C62, C63, C64, C65, C67, C68, C69, C70, C71, D1, D10, D11, D12, D2, D23, D24, D25, D26, D27, D28, D29, D3, D30, D31, D32, D33, D34, D4, D5, D6, D7, D8, D9, R112, R113, R114, R115, R17, R18, R19, R20, R29, R30, R31, R32, R41, R42, R43, R44, R82, R83, R84, R85, R94, R95, R96, R97, U10, U11, U12, U5, U6, U7: moved to F.Cu
- moved C33 224.8 mm to (-49.5, 102.5)
- moved C35 224.8 mm to (-54.2, 95.2)
- moved R100 224.8 mm to (-47.8, 102.5)
- moved R102 224.8 mm to (-46.0, 102.5)
- moved R104 224.8 mm to (-44.2, 102.5)
- moved R110 224.8 mm to (-41.2, 94.5)
- moved R111 224.8 mm to (-42.5, 102.5)
- moved R98 224.8 mm to (-54.2, 97.0)
- moved U26 224.8 mm to (-47.8, 96.2)
- moved C34 223.5 mm to (-48.8, 90.0)
- moved J36 143.2 mm to (-60.0, 62.5)
- moved C10 141.5 mm to (-28.0, 75.2)
- moved C11 141.5 mm to (-24.2, 75.2)
- moved C12 141.5 mm to (-36.5, 52.8)
- moved C13 141.5 mm to (-40.5, 52.8)
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Routing:
- net 5V_IN_15: track 6.35 -> 89.8 mm
- net /AnalogInput/ExternalADC/3V3_IN_21: track 2.25 -> 76.5 mm
- net 5V_IN_16: track 6.49 -> 78.0 mm
- net 10V_IN_6: track 6.35 -> 77.7 mm
- net 5V_IN_10: track 6.24 -> 76.2 mm
- net 5V_IN_1: track 6.24 -> 76.0 mm
- net GND: track 178.0 -> 109.0 mm
- net /AnalogInput/ExternalADC/3V3_IN_22: track 2.00 -> 65.0 mm
- net /AnalogInput/3V3_IN_1: track 2.45 -> 63.6 mm
- net 10V_IN_5: track 6.35 -> 65.9 mm
- net 5V_IN_17: track 6.35 -> 65.8 mm
- net 5V_IN_2: track 6.24 -> 64.3 mm
- net 5V_IN_9: track 6.24 -> 64.0 mm
- net /AnalogInput/3V3_IN_10: track 2.25 -> 59.8 mm
- net /AnalogInput/3V3_IN_20: track 2.25 -> 59.4 mm
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Other:
- board size 250 x 100 mm -> 220 x 145.5 mm

Commit message: More routing
Parts:
- C31: moved to B.Cu
- C33, C34, C35, R100, R102, R104, R110, R111, R98, U26: moved to F.Cu
- moved R110 171.3 mm to (130.0, 89.2), turned to 90 degrees
- moved C33 171.3 mm to (121.2, 89.2), turned to 270 degrees
- moved R100 171.3 mm to (123.0, 89.2), turned to 90 degrees
- moved R102 171.3 mm to (124.8, 89.2), turned to 90 degrees
- moved R104 171.3 mm to (126.5, 89.2), turned to 90 degrees
- moved R111 171.3 mm to (128.2, 89.2), turned to 90 degrees
- moved C34 170.6 mm to (121.5, 100.8)
- moved R98 170.5 mm to (116.2, 93.8)
- moved C35 170.5 mm to (116.2, 97.2)
- moved U26 170.5 mm to (122.8, 95.5)
- moved J23 103.8 mm to (-81.2, 98.5)
- moved J1 103.8 mm to (-81.2, 109.8)
- moved D34 78.5 mm to (82.8, 115.2), turned to 180 degrees
- moved C71 77.8 mm to (82.8, 113.2), turned to 0 degrees
- moved D33 77.0 mm to (82.8, 108.8), turned to 180 degrees
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Connections:
- J28 pad 2: 10V_IN_7 -> 5V_IN_19
- J29 pad 2: 10V_IN_8 -> 5V_IN_20
- J30 pad 2: 10V_IN_9 -> 5V_IN_21
- J31 pad 2: 10V_IN_10 -> 5V_IN_22
- J32 pad 2: 5V_IN_19 -> 10V_IN_7
- J33 pad 2: 5V_IN_20 -> 10V_IN_8
- J34 pad 2: 5V_IN_21 -> 10V_IN_9
- J35 pad 2: 5V_IN_22 -> 10V_IN_10
- U26 pad 19: EADC_ADC_7 -> EADC_ADC_12
- U26 pad 2: EADC_ADC_1 -> EADC_ADC_6
- U26 pad 20: EADC_ADC_8 -> EADC_ADC_11
- U26 pad 21: EADC_ADC_9 -> EADC_ADC_10
- U26 pad 22: EADC_ADC_10 -> EADC_ADC_9
- U26 pad 3: EADC_ADC_2 -> EADC_ADC_5
- U26 pad 31: EADC_ADC_11 -> EADC_ADC_8
- U26 pad 32: EADC_ADC_12 -> EADC_ADC_7
- U26 pad 4: EADC_ADC_3 -> EADC_ADC_4
- U26 pad 5: EADC_ADC_4 -> EADC_ADC_3
- U26 pad 6: EADC_ADC_5 -> EADC_ADC_2
- U26 pad 7: EADC_ADC_6 -> EADC_ADC_1
Routing:
- net /AnalogInput/ExternalADC/3V3_IN_32: track 2.25 -> 111.2 mm
- net /AnalogInput/ExternalADC/3V3_IN_31: track 2.25 -> 102.8 mm
- net /AnalogInput/ExternalADC/3V3_IN_30: track 2.25 -> 91.4 mm
- net 10V_IN_10: track 6.35 -> 91.3 mm
- net 10V_IN_9: track 6.35 -> 79.6 mm
- net /AnalogInput/3V3_IN_11: track 43.6 -> 105.1 mm
- net /AnalogInput/3V3_IN_10: track 59.8 -> 120.9 mm
- net 10V_IN_8: track 6.35 -> 67.0 mm
- net /AnalogInput/3V3_IN_9: track 47.6 -> 106.8 mm
- net /AnalogInput/ExternalADC/3V3_IN_29: track 19.2 -> 77.5 mm
- net /AnalogInput/3V3_IN_12: track 37.6 -> 95.6 mm
- net EADC_ADC_12: track 0.00 -> 57.8 mm
- net EADC_ADC_1: track 0.00 -> 57.3 mm
- net /AnalogInput/3V3_IN_18: track 35.1 -> 85.3 mm
- net /AnalogInput/3V3_IN_19: track 47.3 -> 96.0 mm
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- added copper zone on F.Cu, net GND

Commit message: Routing
Parts:
- added G***: LOGO, PCB_Morro_Bay:P_Logo, B.Cu at (147.2, 37.2)
- added G***: LOGO, PCB_Morro_Bay:J_Logo, B.Cu at (209.0, 37.5)
- added G***: LOGO, PCB_Morro_Bay:Logo, B.Cu at (186.8, 123.0)
- C1, C2, C6, C9, D35, D36, JP1, R1, R116, R117, R2, R3, R4, R5, R6, R7, R8, TP1, TP2, TP3, TP4, U1, U13, U2, Y1: moved to F.Cu
- C12, C20, C21, C22, C23, C24, C25, C26, C30, C32, C40, C41, C66, C67, FB2: moved to B.Cu
- Y3: footprint Crystal:Crystal_SMD_SeikoEpson_MC146-4Pin_6.7x1.5mm_HandSoldering -> PCB_Morro_Bay:Crystal_Epson_MC-146
- moved C11 145.6 mm to (121.0, 84.8), turned to 90 degrees
- moved C12 141.7 mm to (102.8, 78.8)
- moved D22 140.6 mm to (70.5, 113.5), turned to 270 degrees
- moved R70 138.4 mm to (68.8, 113.5), turned to 90 degrees
- moved D21 137.9 mm to (70.5, 109.0), turned to 270 degrees
- moved FB2 137.4 mm to (102.8, 81.2), turned to 180 degrees
- moved R69 135.7 mm to (68.8, 109.0), turned to 90 degrees
- moved TP6 134.5 mm to (65.5, 113.5), turned to 0 degrees
- moved TP5 131.7 mm to (65.5, 109.0), turned to 180 degrees
- moved Y2 129.7 mm to (109.5, 85.0)
- moved C14 126.7 mm to (79.5, 73.5)
- moved C10 126.6 mm to (98.2, 84.8), turned to 270 degrees
- moved Y3 125.1 mm to (81.8, 71.2), turned to 0 degrees
- moved C20 125.1 mm to (97.0, 80.5), turned to 90 degrees
- moved C21 125.1 mm to (99.0, 80.5), turned to 90 degrees
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Routing:
- net +3V3: track 19.8 -> 1200.1 mm, vias 0 -> 23
- net +5V: track 0.00 -> 1154.1 mm, vias 0 -> 18
- net GND: track 109.2 -> 275.1 mm, vias 0 -> 208
- net SAMD_ADC_20: track 4.16 -> 131.0 mm
- net SAMD_ADC_19: track 4.16 -> 116.9 mm
- net SAMD_ADC_13: track 2.16 -> 108.6 mm
- net SAMD_ADC_17: track 4.16 -> 106.9 mm
- net SAMD_ADC_16: track 2.16 -> 104.3 mm
- net SAMD_ADC_18: track 4.16 -> 101.3 mm
- net SAMD_ADC_14: track 2.16 -> 98.7 mm
- net SAMD_ADC_15: track 2.16 -> 94.2 mm
- net SAMD_ADC_12: track 4.16 -> 95.7 mm
- net /GPIO_4: track 0.00 -> 80.6 mm, vias 0 -> 3
- net SAMD_ADC_11: track 4.16 -> 81.5 mm
- net /USB_D+: track 8.33 -> 85.7 mm, vias 0 -> 2
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- added copper zone on B.Cu, net +3V3
- added copper zone on F.Cu, net +3V3
- added copper zone on B.Cu, net +5V
- added copper zone on F.Cu, net +5V
- added copper zone on F.Cu, net /VIN
- added copper zone on B.Cu, net GND
- added copper zone on F.Cu, net Net-(C28-Pad1)
Other:
- board text added: "Designed by Jasper Rubin in 2020"
- board text added: "Morro Bay Data Acquisition Board"
